Commit message: New node emotion.py

File: install/my_robot_sim/share/my_robot_sim/urdf/my_robot.urdf (robot description, URDF)
Before this commit: robot rsc, 10 links, 9 joints
Links:
- link screen: geometry collision mesh filename=package://my_robot_sim/meshes/screen.STL scale=0.01 0.01 0.01; visual mesh filename=package://my_robot_sim/meshes/screen.STL scale=0.01 0.01 0.01
Joints:
- joint base_to_body: axis 0 0 1 -> (none); limit lower=-1.57 upper=1.57 effort=50 velocity=5.0 -> (none); type revolute -> fixed
- joint screen_to_body: parent cornice -> base_link
