Commit message: Third motion of the robot

File: src/my_robot_sim/urdf/my_robot.urdf (robot description, URDF)
Before this commit: robot rsc, 10 links, 9 joints
Joints:
- joint base_to_body: axis (none) -> 0 0 1; limit (none) -> lower=-1.57 upper=1.57 effort=100 velocity=1.0; type fixed -> revolute

Commit message: movements with right duration and body motion

File: src/my_robot_sim/urdf/my_robot.urdf (robot description, URDF)
Before this commit: robot rsc, 10 links, 9 joints
Joints:
- joint base_to_body: axis 0 0 1 -> (none); limit lower=-1.57 upper=1.57 effort=100 velocity=1.0 -> (none); type revolute -> fixed

Commit message: renaming

File: src/my_robot_sim/urdf/my_robot.urdf (robot description, URDF)
Before this commit: robot rsc, 10 links, 9 joints
Links:
- removed link arm_1
- removed link arm_2
- removed link base_link
- removed link cornice
- removed link piattello
- added link body; collision mesh filename=package://my_robot_sim/meshes/body.STL scale=0.01 0.01 0.01; visual mesh filename=package://my_robot_sim/meshes/body.STL scale=0.01 0.01 0.01
- added link flipper_l; collision mesh filename=package://my_robot_sim/meshes/flipper.STL scale=0.01 0.01 0.01; visual mesh filename=package://my_robot_sim/meshes/flipper.STL scale=0.01 0.01 0.01
- added link flipper_r; collision mesh filename=package://my_robot_sim/meshes/flipper.STL scale=0.01 0.01 0.01; visual mesh filename=package://my_robot_sim/meshes/flipper.STL scale=0.01 0.01 0.01
- added link frame; collision mesh filename=package://my_robot_sim/meshes/frame.STL scale=0.01 0.01 0.01; visual mesh filename=package://my_robot_sim/meshes/frame.STL scale=0.01 0.01 0.01
- added link lid; collision mesh filename=package://my_robot_sim/meshes/lid.STL scale=0.01 0.01 0.01; visual mesh filename=package://my_robot_sim/meshes/lid.STL scale=0.01 0.01 0.01
Joints:
- removed joint arm1_to_pivot
- removed joint arm2_to_pivot
- removed joint cornice_to_body
- removed joint piattello_to_body
- added joint flipper_l_to_body: type continuous, parent body, child flipper_l, origin xyz=0 0.05 0.9 rpy=0 0 0, axis 1 0 0
- added joint flipper_r_to_body: type continuous, parent body, child flipper_r, origin xyz=0 0.05 0.9 rpy=0 0 0, axis 1 0 0
- added joint frame_to_body: type fixed, parent body, child frame, origin xyz=0 0 0 rpy=0 0 0
- added joint lid_to_body: type fixed, parent body, child lid, origin xyz=0 0 0 rpy=0 0 0
- joint back_to_body: parent base_link -> body
- joint base_to_body: child base_link -> body
- joint button_to_body: parent base_link -> body
- joint image_to_body: parent base_link -> body
- joint screen_to_body: parent base_link -> body
