Commit message: renaming package

File: src/my_robot_sim/urdf/my_robot.urdf.xacro (robot description, xacro)
@@ -1,6 +1,6 @@
 <?xml version="1.0" encoding="utf-8"?>
 <robot name="rsc" xmlns:xacro="http://www.ros.org/wiki/xacro">
- <xacro:property name="button_color" value="yellow"/>
- <xacro:property name="face" value="joy"/>
+ <xacro:property name="button_color" value="yellow"/>   <!-- Modify here the color of the botton -->
+ <xacro:property name="face" value="joy"/>   <!-- Modify here the emotion face of the RSC -->
   <!-- Define materials -->
 <material name="blue">
